File: LedStrip/Hardware/esp-ws2812.sch (KiCad schematic (older format))
At the start: 11 parts, among them P3 CONN_01X01, P4 CONN_01X02, Q1 BSS138, U1 MCP1700, U2 ESP-01v090

Commit message: finished up the layout of the board
Parts:
- C1: value C -> 0.1uf; Comments (none) -> a cap of around 0.1 to 10 uf - anything in that range will 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
- C2: value CP -> 2.2uf; Notes (none) -> a Tant cap in the 1-10uf range - anything that fits will do
- C3: value C -> 0.1uf; Notes (none) -> Any cap in the 0.1-10uf range
- C4: value CP -> 2.2uf; Notes (none) -> Any tant cap in the 1-10uf range - what ever fits will do
Changed lines of the file:
@@
 LIBS:valves
 LIBS:ESP8266
-LIBS:espbase-cache
+LIBS:esp-ws2812-cache
 EELAYER 25 0
 EELAYER END
@@
 P 1750 2100
 F 0 "C1" H 1775 2200 50  0000 L CNN
-F 1 "C" H 1775 2000 50  0000 L CNN
+F 1 "0.1uf" H 1775 2000 50  0000 L CNN
 F 2 "Capacitors_SMD:C_0805_HandSoldering" H 1788 1950 50  0001 C CNN
 F 3 "" H 1750 2100 50  0000 C CNN
+F 4 "a  cap of around 0.1 to 10 uf - anything in that range will do" H 1750 2100 60  0001 C CNN "Comments"
 	1    1750 2100
 	1    0    0    -1
@@
 P 2000 2100
 F 0 "C2" H 2025 2200 50  0000 L CNN
-F 1 "CP" H 2025 2000 50  0000 L CNN
+F 1 "2.2uf" H 2025 2000 50  0000 L CNN
 F 2 "SMD_Packages:SMD-1210_Pol" H 2038 1950 50  0001 C CNN
 F 3 "" H 2000 2100 50  0000 C CNN
+F 4 "a Tant cap in the 1-10uf range - anything that fits will do" H 2000 2100 60  0001 C CNN "Notes"
 	1    2000 2100
 	1    0    0    -1
@@
 P 2950 2100
 F 0 "C3" H 2975 2200 50  0000 L CNN
-F 1 "C" H 2975 2000 50  0000 L CNN
+F 1 "0.1uf" H 2975 2000 50  0000 L CNN
 F 2 "Capacitors_SMD:C_0805_HandSoldering" H 2988 1950 50  0001 C CNN
 F 3 "" H 2950 2100 50  0000 C CNN
+F 4 "Any cap in the 0.1-10uf range" H 2950 2100 60  0001 C CNN "Notes"
 	1    2950 2100
 	1    0    0    -1
@@
 P 3200 2100
 F 0 "C4" H 3225 2200 50  0000 L CNN
-F 1 "CP" H 3225 2000 50  0000 L CNN
+F 1 "2.2uf" H 3225 2000 50  0000 L CNN
 F 2 "SMD_Packages:SMD-1210_Pol" H 3238 1950 50  0001 C CNN
 F 3 "" H 3200 2100 50  0000 C CNN
+F 4 "Any tant cap in the 1-10uf range - what ever fits will do" H 3200 2100 60  0001 C CNN "Notes"
 	1    3200 2100
 	1    0    0    -1

Commit message: new circuit board with power passthru
Parts:
- added C5: 1000uf, Discret:CP6, symbol CP
- added P1: CONN_01X02, Pin_Headers:Pin_Header_Straight_1x02, symbol CONN_01X02
- C2: footprint SMD_Packages:SMD-1210_Pol -> Capacitors_Tantalum_SMD:TantalC_SizeD_EIA-7343_HandSoldering
Connections:
- net +5V: now also C5.1, P1.2 (P2)
- net GND: now also C5.2, P1.1 (P1)
Changed lines of the file:
@@
 $EndComp
 $Comp
-L +5V #PWR01
+L +5V #PWR5
 U 1 1 580E0F63
 P 1550 1850
-F 0 "#PWR01" H 1550 1700 50  0001 C CNN
+F 0 "#PWR5" H 1550 1700 50  0001 C CNN
 F 1 "+5V" H 1550 1990 50  0000 C CNN
 F 2 "" H 1550 1850 50  0000 C CNN
@@
 $EndComp
 $Comp
-L GND #PWR02
+L GND #PWR6
 U 1 1 580E0F79
 P 1550 2350
-F 0 "#PWR02" H 1550 2100 50  0001 C CNN
+F 0 "#PWR6" H 1550 2100 50  0001 C CNN
 F 1 "GND" H 1550 2200 50  0000 C CNN
 F 2 "" H 1550 2350 50  0000 C CNN
@@
 F 0 "C2" H 2025 2200 50  0000 L CNN
 F 1 "2.2uf" H 2025 2000 50  0000 L CNN
-F 2 "SMD_Packages:SMD-1210_Pol" H 2038 1950 50  0001 C CNN
+F 2 "Capacitors_Tantalum_SMD:TantalC_SizeD_EIA-7343_HandSoldering" H 2038 1950 50  0001 C CNN
 F 3 "" H 2000 2100 50  0000 C CNN
 F 4 "a Tant cap in the 1-10uf range - anything that fits will do" H 2000 2100 60  0001 C CNN "Notes"
@@
 $EndComp
 $Comp
-L +3.3V #PWR03
+L +3.3V #PWR10
 U 1 1 580E1212
 P 3550 1800
-F 0 "#PWR03" H 3550 1650 50  0001 C CNN
+F 0 "#PWR10" H 3550 1650 50  0001 C CNN
 F 1 "+3.3V" H 3550 1940 50  0000 C CNN
 F 2 "" H 3550 1800 50  0000 C CNN
@@
 Connection ~ 1750 1950
 $Comp
-L +3.3V #PWR04
+L +3.3V #PWR12
 U 1 1 580E14E4
 P 4600 2400
-F 0 "#PWR04" H 4600 2250 50  0001 C CNN
+F 0 "#PWR12" H 4600 2250 50  0001 C CNN
 F 1 "+3.3V" H 4600 2540 50  0000 C CNN
 F 2 "" H 4600 2400 50  0000 C CNN
@@
 Connection ~ 4600 2250
 $Comp
-L GND #PWR05
+L GND #PWR13
 U 1 1 580E154C
 P 6800 1800
-F 0 "#PWR05" H 6800 1550 50  0001 C CNN
+F 0 "#PWR13" H 6800 1550 50  0001 C CNN
 F 1 "GND" H 6800 1650 50  0000 C CNN
 F 2 "" H 6800 1800 50  0000 C CNN
@@
 GPIO2_5
 $Comp
-L +3.3V #PWR06
+L +3.3V #PWR9
 U 1 1 580E1E4B
 P 3050 2750
-F 0 "#PWR06" H 3050 2600 50  0001 C CNN
+F 0 "#PWR9" H 3050 2600 50  0001 C CNN
 F 1 "+3.3V" H 3050 2890 50  0000 C CNN
 F 2 "" H 3050 2750 50  0000 C CNN
@@
 $EndComp
 $Comp
-L +5V #PWR07
+L +5V #PWR11
 U 1 1 580E1EC9
 P 3650 2750
-F 0 "#PWR07" H 3650 2600 50  0001 C CNN
+F 0 "#PWR11" H 3650 2600 50  0001 C CNN
 F 1 "+5V" H 3650 2890 50  0000 C CNN
 F 2 "" H 3650 2750 50  0000 C CNN
@@
 $EndComp
 $Comp
-L +5V #PWR08
+L +5V #PWR7
 U 1 1 580E1FBD
 P 1900 2950
-F 0 "#PWR08" H 1900 2800 50  0001 C CNN
+F 0 "#PWR7" H 1900 2800 50  0001 C CNN
 F 1 "+5V" H 1900 3090 50  0000 C CNN
 F 2 "" H 1900 2950 50  0000 C CNN
@@
 $EndComp
 $Comp
-L GND #PWR09
+L GND #PWR8
 U 1 1 580E1FEF
 P 2100 2950
-F 0 "#PWR09" H 2100 2700 50  0001 C CNN
+F 0 "#PWR8" H 2100 2700 50  0001 C CNN
 F 1 "GND" H 2100 2800 50  0000 C CNN
 F 2 "" H 2100 2950 50  0000 C CNN
@@
 Wire Wire Line
 	1900 2950 1900 3100
+$Comp
+L CP C5
+U 1 1 5810336B
+P 950 2100
+F 0 "C5" H 975 2200 50  0000 L CNN
+F 1 "1000uf" H 975 2000 50  0000 L CNN
+F 2 "Discret:CP6" H 988 1950 50  0001 C CNN
+F 3 "" H 950 2100 50  0000 C CNN
+F 4 "Basically a big cap for powering lights" H 950 2100 60  0001 C CNN "Notes"
+	1    950  2100
+	1    0    0    -1
+$EndComp
+$Comp
+L +5V #PWR1
+U 1 1 58103426
+P 950 1850
+F 0 "#PWR1" H 950 1700 50  0001 C CNN
+F 1 "+5V" H 950 1990 50  0000 C CNN
+F 2 "" H 950 1850 50  0000 C CNN
+F 3 "" H 950 1850 50  0000 C CNN
+	1    950  1850
+	1    0    0    -1
+$EndComp
+$Comp
+L GND #PWR2
+U 1 1 58103455
+P 950 2350
+F 0 "#PWR2" H 950 2100 50  0001 C CNN
+F 1 "GND" H 950 2200 50  0000 C CNN
+F 2 "" H 950 2350 50  0000 C CNN
+F 3 "" H 950 2350 50  0000 C CNN
+	1    950  2350
+	1    0    0    -1
+$EndComp
+Wire Wire Line
+	950  1950 950  1850
+Wire Wire Line
+	950  2350 950  2250
+$Comp
+L CONN_01X02 P1
+U 1 1 5810362E
+P 1250 3300
+F 0 "P1" H 1250 3450 50  0000 C CNN
+F 1 "CONN_01X02" V 1350 3300 50  0000 C CNN
+F 2 "Pin_Headers:Pin_Header_Straight_1x02" H 1250 3300 50  0001 C CNN
+F 3 "" H 1250 3300 50  0000 C CNN
+	1    1250 3300
+	0    1    1    0
+$EndComp
+$Comp
+L +5V #PWR3
+U 1 1 58103634
+P 1200 2950
+F 0 "#PWR3" H 1200 2800 50  0001 C CNN
+F 1 "+5V" H 1200 3090 50  0000 C CNN
+F 2 "" H 1200 2950 50  0000 C CNN
+F 3 "" H 1200 2950 50  0000 C CNN
+	1    1200 2950
+	1    0    0    -1
+$EndComp
+$Comp
+L GND #PWR4
+U 1 1 5810363A
+P 1400 2950
+F 0 "#PWR4" H 1400 2700 50  0001 C CNN
+F 1 "GND" H 1400 2800 50  0000 C CNN
+F 2 "" H 1400 2950 50  0000 C CNN
+F 3 "" H 1400 2950 50  0000 C CNN
+	1    1400 2950
+	0    -1   -1   0
+$EndComp
+Wire Wire Line
+	1400 2950 1300 2950
+Wire Wire Line
+	1300 2950 1300 3100
+Wire Wire Line
+	1200 2950 1200 3100
 $EndSCHEMATC

Commit message: board update
Parts:
- C2: footprint Capacitors_Tantalum_SMD:TantalC_SizeD_EIA-7343_HandSoldering -> SMD_Packages:SMD-1210_Pol
- C5: footprint Discret:CP6 -> Capacitors_ThroughHole:C_Radial_D6.3_L11.2_P2.5
Changed lines of the file:
@@
 $EndComp
 $Comp
-L +5V #PWR5
+L +5V #PWR01
 U 1 1 580E0F63
 P 1550 1850
-F 0 "#PWR5" H 1550 1700 50  0001 C CNN
+F 0 "#PWR01" H 1550 1700 50  0001 C CNN
 F 1 "+5V" H 1550 1990 50  0000 C CNN
 F 2 "" H 1550 1850 50  0000 C CNN
@@
 $EndComp
 $Comp
-L GND #PWR6
+L GND #PWR02
 U 1 1 580E0F79
 P 1550 2350
-F 0 "#PWR6" H 1550 2100 50  0001 C CNN
+F 0 "#PWR02" H 1550 2100 50  0001 C CNN
 F 1 "GND" H 1550 2200 50  0000 C CNN
 F 2 "" H 1550 2350 50  0000 C CNN
@@
 F 0 "C2" H 2025 2200 50  0000 L CNN
 F 1 "2.2uf" H 2025 2000 50  0000 L CNN
-F 2 "Capacitors_Tantalum_SMD:TantalC_SizeD_EIA-7343_HandSoldering" H 2038 1950 50  0001 C CNN
+F 2 "SMD_Packages:SMD-1210_Pol" H 2038 1950 50  0001 C CNN
 F 3 "" H 2000 2100 50  0000 C CNN
 F 4 "a Tant cap in the 1-10uf range - anything that fits will do" H 2000 2100 60  0001 C CNN "Notes"
@@
 $EndComp
 $Comp
-L +3.3V #PWR10
+L +3.3V #PWR03
 U 1 1 580E1212
 P 3550 1800
-F 0 "#PWR10" H 3550 1650 50  0001 C CNN
+F 0 "#PWR03" H 3550 1650 50  0001 C CNN
 F 1 "+3.3V" H 3550 1940 50  0000 C CNN
 F 2 "" H 3550 1800 50  0000 C CNN
@@
 Connection ~ 1750 1950
 $Comp
-L +3.3V #PWR12
+L +3.3V #PWR04
 U 1 1 580E14E4
 P 4600 2400
-F 0 "#PWR12" H 4600 2250 50  0001 C CNN
+F 0 "#PWR04" H 4600 2250 50  0001 C CNN
 F 1 "+3.3V" H 4600 2540 50  0000 C CNN
 F 2 "" H 4600 2400 50  0000 C CNN
@@
 Connection ~ 4600 2250
 $Comp
-L GND #PWR13
+L GND #PWR05
 U 1 1 580E154C
 P 6800 1800
-F 0 "#PWR13" H 6800 1550 50  0001 C CNN
+F 0 "#PWR05" H 6800 1550 50  0001 C CNN
 F 1 "GND" H 6800 1650 50  0000 C CNN
 F 2 "" H 6800 1800 50  0000 C CNN
@@
 GPIO2_5
 $Comp
-L +3.3V #PWR9
+L +3.3V #PWR06
 U 1 1 580E1E4B
 P 3050 2750
-F 0 "#PWR9" H 3050 2600 50  0001 C CNN
+F 0 "#PWR06" H 3050 2600 50  0001 C CNN
 F 1 "+3.3V" H 3050 2890 50  0000 C CNN
 F 2 "" H 3050 2750 50  0000 C CNN
@@
 $EndComp
 $Comp
-L +5V #PWR11
+L +5V #PWR07
 U 1 1 580E1EC9
 P 3650 2750
-F 0 "#PWR11" H 3650 2600 50  0001 C CNN
+F 0 "#PWR07" H 3650 2600 50  0001 C CNN
 F 1 "+5V" H 3650 2890 50  0000 C CNN
 F 2 "" H 3650 2750 50  0000 C CNN
@@
 $EndComp
 $Comp
-L +5V #PWR7
+L +5V #PWR08
 U 1 1 580E1FBD
 P 1900 2950
-F 0 "#PWR7" H 1900 2800 50  0001 C CNN
+F 0 "#PWR08" H 1900 2800 50  0001 C CNN
 F 1 "+5V" H 1900 3090 50  0000 C CNN
 F 2 "" H 1900 2950 50  0000 C CNN
@@
 $EndComp
 $Comp
-L GND #PWR8
+L GND #PWR09
 U 1 1 580E1FEF
 P 2100 2950
-F 0 "#PWR8" H 2100 2700 50  0001 C CNN
+F 0 "#PWR09" H 2100 2700 50  0001 C CNN
 F 1 "GND" H 2100 2800 50  0000 C CNN
 F 2 "" H 2100 2950 50  0000 C CNN
@@
 F 0 "C5" H 975 2200 50  0000 L CNN
 F 1 "1000uf" H 975 2000 50  0000 L CNN
-F 2 "Discret:CP6" H 988 1950 50  0001 C CNN
+F 2 "Capacitors_ThroughHole:C_Radial_D6.3_L11.2_P2.5" H 988 1950 50  0001 C CNN
 F 3 "" H 950 2100 50  0000 C CNN
 F 4 "Basically a big cap for powering lights" H 950 2100 60  0001 C CNN "Notes"
@@
 $EndComp
 $Comp
-L +5V #PWR1
+L +5V #PWR010
 U 1 1 58103426
 P 950 1850
-F 0 "#PWR1" H 950 1700 50  0001 C CNN
+F 0 "#PWR010" H 950 1700 50  0001 C CNN
 F 1 "+5V" H 950 1990 50  0000 C CNN
 F 2 "" H 950 1850 50  0000 C CNN
@@
 $EndComp
 $Comp
-L GND #PWR2
+L GND #PWR011
 U 1 1 58103455
 P 950 2350
-F 0 "#PWR2" H 950 2100 50  0001 C CNN
+F 0 "#PWR011" H 950 2100 50  0001 C CNN
 F 1 "GND" H 950 2200 50  0000 C CNN
 F 2 "" H 950 2350 50  0000 C CNN
@@
 $EndComp
 $Comp
-L +5V #PWR3
+L +5V #PWR012
 U 1 1 58103634
 P 1200 2950
-F 0 "#PWR3" H 1200 2800 50  0001 C CNN
+F 0 "#PWR012" H 1200 2800 50  0001 C CNN
 F 1 "+5V" H 1200 3090 50  0000 C CNN
 F 2 "" H 1200 2950 50  0000 C CNN
@@
 $EndComp
 $Comp
-L GND #PWR4
+L GND #PWR013
 U 1 1 5810363A
 P 1400 2950
-F 0 "#PWR4" H 1400 2700 50  0001 C CNN
+F 0 "#PWR013" H 1400 2700 50  0001 C CNN
 F 1 "GND" H 1400 2800 50  0000 C CNN
 F 2 "" H 1400 2950 50  0000 C CNN

Commit message: added a uart/gpio0 interface to the esp board
Parts:
- added P2: CONN_01X04, Pin_Headers:Pin_Header_Straight_1x04, symbol CONN_01X04
Connections:
- net GND: now also P2.1 (P1)
- net GPIO0: now also P2.3 (P3)
- net RX: now also P2.4 (P4)
- net TX: now also P2.2 (P2)
Changed lines of the file:
@@
 Wire Wire Line
 	1200 2950 1200 3100
+$Comp
+L CONN_01X04 P2
+U 1 1 58156601
+P 1450 4550
+F 0 "P2" H 1450 4800 50  0000 C CNN
+F 1 "CONN_01X04" V 1550 4550 50  0000 C CNN
+F 2 "Pin_Headers:Pin_Header_Straight_1x04" H 1450 4550 50  0001 C CNN
+F 3 "" H 1450 4550 50  0000 C CNN
+	1    1450 4550
+	0    1    1    0
+$EndComp
+$Comp
+L GND #PWR014
+U 1 1 581566D2
+P 1700 4200
+F 0 "#PWR014" H 1700 3950 50  0001 C CNN
+F 1 "GND" H 1700 4050 50  0000 C CNN
+F 2 "" H 1700 4200 50  0000 C CNN
+F 3 "" H 1700 4200 50  0000 C CNN
+	1    1700 4200
+	0    -1   -1   0
+$EndComp
+Text GLabel 1200 4200 0    60   Input ~ 0
+RX
+Text GLabel 1600 4000 2    60   Input ~ 0
+TX
+Text GLabel 1300 4000 0    60   Input ~ 0
+GPIO0
+Wire Wire Line
+	1300 4000 1400 4000
+Wire Wire Line
+	1400 4000 1400 4350
+Wire Wire Line
+	1200 4200 1300 4200
+Wire Wire Line
+	1300 4200 1300 4350
+Wire Wire Line
+	1700 4200 1600 4200
+Wire Wire Line
+	1600 4200 1600 4350
+Wire Wire Line
+	1600 4000 1500 4000
+Wire Wire Line
+	1500 4000 1500 4350
 $EndSCHEMATC

Commit message: attributions to sparkfun
Other:
- note added: "Level shifter circuit here is a copy of the level shifter in the sparkfun bi-directional level shifter\navailable at https://www.sparkfun.com/products/12009"
Changed lines of the file:
@@
 Wire Wire Line
 	1500 4000 1500 4350
+Text Notes 2600 4000 0    60   ~ 0
+Level shifter circuit here is a copy of the level shifter in the sparkfun bi-directional level shifter\navailable at https://www.sparkfun.com/products/12009
 $EndSCHEMATC

Commit message: small board update for metric tant layouts
Parts:
- C2, C4: footprint SMD_Packages:SMD-1210_Pol -> Capacitors_Tantalum_SMD:TantalC_SizeB_EIA-3528_Wave
Changed lines of the file:
@@
 F 0 "C2" H 2025 2200 50  0000 L CNN
 F 1 "2.2uf" H 2025 2000 50  0000 L CNN
-F 2 "SMD_Packages:SMD-1210_Pol" H 2038 1950 50  0001 C CNN
+F 2 "Capacitors_Tantalum_SMD:TantalC_SizeB_EIA-3528_Wave" H 2038 1950 50  0001 C CNN
 F 3 "" H 2000 2100 50  0000 C CNN
 F 4 "a Tant cap in the 1-10uf range - anything that fits will do" H 2000 2100 60  0001 C CNN "Notes"
@@
 F 0 "C4" H 3225 2200 50  0000 L CNN
 F 1 "2.2uf" H 3225 2000 50  0000 L CNN
-F 2 "SMD_Packages:SMD-1210_Pol" H 3238 1950 50  0001 C CNN
+F 2 "Capacitors_Tantalum_SMD:TantalC_SizeB_EIA-3528_Wave" H 3238 1950 50  0001 C CNN
 F 3 "" H 3200 2100 50  0000 C CNN
 F 4 "Any tant cap in the 1-10uf range - what ever fits will do" H 3200 2100 60  0001 C CNN "Notes"
