File: IRRemote/irremote.sch (KiCad schematic (older format))
At the start: 22 parts, among them P1 USB_OTG, P2 TL1838_PINHEADER, P3 DS18B20_PINHEADER_TO92, Q1 Q_NPN_BEC (MMBT2222ALT1G, 145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, Q2 Q_NPN_BEC (MMBT2222ALT1G, 145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, Q3 Q_NPN_BEC (MMBT2222ALT1G, 145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, Q4 Q_NPN_BEC (MMBT2222ALT1G, 145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, U1 ESP-12E, U2 AP1117

Commit message: board layout complete
Parts:
- removed D1, D2, D3, D4: LED, LEDs:LED-5MM, symbol LED
- added C5: C, Capacitors_SMD:C_0805_HandSoldering, symbol C
- added P4: CONN_02X04, Pin_Headers:Pin_Header_Straight_2x04, symbol CONN_02X04
- added P5, P7: CONN_01X04, Pin_Headers:Pin_Header_Straight_1x04, symbol CONN_01X04
- added P6: CONN_01X05, Pin_Headers:Pin_Header_Straight_1x05, symbol CONN_01X05
- added P8: TEMP6000, Pin_Headers:Pin_Header_Straight_1x03, symbol CONN_01X03
- added P9: CONN_01X02, Pin_Headers:Pin_Header_Straight_1x02, symbol CONN_01X02
- added R10, R11, R12, R8, R9: 4.7k, Resistors_SMD:R_0805_HandSoldering, symbol R
- added R6, R7: 27, Resistors_SMD:R_0805_HandSoldering, symbol R
- added SW1, SW2: SW_PUSH, Buttons_Switches_SMD:SW_SPST_EVQPE1, symbol SW_PUSH
- added U3: FT230XS, Housings_SSOP:SSOP-16_3.9x4.9mm_Pitch0.635mm, symbol FT230XS
- C1, C4: footprint Capacitors_Tantalum_SMD:TantalC_SizeB_EIA-3528_Wave -> Capacitors_Tantalum_SMD:TantalC_SizeB_EIA-3528_Reflow
Connections:
- net +3V3: now also P5.4 (P4), P8.1 (P1), R11.1, R12.1, R8.2, R9.2
- net +5V: now also P9.1 (P1), U3.12 (VCC)
- net GND: now also C5.1, P5.1 (P1), P8.2 (P2), P9.2 (P2), R10.1, SW1.2, SW2.1, U3.13 (GND), U3.5 (GND)
- net at U1.1 (REST): now also R8.1, SW1.1
- net at U1.10 (MISO): now also P7.3 (P3)
- net at U1.11 (GPIO9): now also P6.1 (P1)
- net at U1.12 (GPIO10): now also P6.2 (P2)
- net at U1.13 (MOSI): now also P7.2 (P2)
- net at U1.14 (SCLK): now also P7.1 (P1)
- net at U1.16 (GPIO15): now also R10.2
- net at U1.17 (GPIO2): now also R11.2
- net at U1.18 (GPIO0): now also R12.2, SW2.2
- net TEMT: now reaches U1.2 (ADC)
- net TEMT: now also P8.3 (P3)
- net TXD_UA_1: now reaches U1.21 (RXD)
- net TXD_UA_1: now also P5.3 (P3), U3.1 (TXD)
- net RXD_UA_1: now reaches U1.22 (TXD)
- net RXD_UA_1: now also P5.2 (P2), U3.4 (RXD)
- net at U1.3 (CH_PD): now also R9.1
- net at U1.4 (GPIO16): now also P6.5 (P5)
- net at U1.5 (GPIO14): now also P6.4 (P4)
- net at U1.7 (GPIO13): now also P6.3 (P3)
- net at U1.9 (CS0): now also P7.4 (P4)
- net USBDM_1_N: now reaches P1.2 (D-)
- net USBDM_1_N: now also R7.1
- net USBDP_1_P: now reaches P1.3 (D+)
- net USBDP_1_P: now also R6.2
- net LED_DR_5: now reaches Q1.3 (C), Q2.3 (C), Q3.3 (C), Q4.3 (C)
- net LED_DR_5: now also P4.1 (P1), P4.3 (P3), P4.5 (P5), P4.7 (P7)
- net at R1.2: now also P4.4 (P4)
- net at R2.2: now also P4.6 (P6)
- net at R4.2: now also P4.2 (P2)
- net at R5.2: now also P4.8 (P8)
- new net: C5.2, U3.10 (3V3OUT), U3.11 (RESET), U3.3 (VCCIO)
- new net: U3.2 (RTS), U3.6 (CTS)
- new net: R6.1, U3.8 (USBDP)
- new net: R7.2, U3.9 (USBDM)
Other:
- moved on the sheet: C1, C2, C3, C4, P1, P2, P3, Q2, R1, R2, R3, R4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
