File: IRRemote/hardware/irremote.kicad_pcb (KiCad board)
At the start: 2 copper layers, 68.5 x 32 mm, 41 parts, among them P1 USB_OTG, P2 TL1838_PINHEADER, P3 DS18B20_PINHEADER_TO92, P4 CONN_02X04, P5 CONN_01X04, P6 CONN_01X05, P7 CONN_01X04, P8 TEMP6000, P9 CONN_01X02, Q1 Q_NPN_BEC (MMBT2222ALT1G, 145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

Commit message: 3d view of board
Other:
- board text added: "+3.3"
- board text added: "+5"
- board text added: "GND"
- board text added: "GPIO"
- board text added: "IR IN"
- board text added: "IR OUT x 4"
- board text added: "LIGHT"
- board text added: "PROG"
- board text added: "RESET"
- board text added: "RX"
- board text added: "TEMP"
- board text added: "TX"
Changed lines of the file:
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@@
     (area 100.024999 47.534523 180.387584 87.6525)
     (thickness 1.6)
-    (drawings 5)
+    (drawings 22)
     (tracks 455)
     (zones 0)
@@
   (page A4)
   (layers
-    (0 F.Cu signal hide)
-    (31 B.Cu signal hide)
+    (0 F.Cu signal)
+    (31 B.Cu signal)
     (32 B.Adhes user)
     (33 F.Adhes user)
@@
     (46 B.CrtYd user)
     (47 F.CrtYd user)
-    (48 B.Fab user)
+    (48 B.Fab user hide)
     (49 F.Fab user hide)
   )
@@
     (descr "Through hole pin header")
     (tags "pin header")
-    (fp_text reference P5 (at 2.404 -0.7705 360) (layer F.SilkS)
+    (fp_text reference P5 (at -2.1045 3.2935 360) (layer F.SilkS)
       (effects (font (size 1 1) (thickness 0.15)))
     )
@@
     (descr "Light Touch Switch")
     (attr smd)
-    (fp_text reference SW2 (at -0.154 2.423) (layer F.SilkS)
+    (fp_text reference SW2 (at 0.0365 0.2005) (layer F.SilkS)
       (effects (font (size 1 1) (thickness 0.15)))
     )
@@
     (descr "Light Touch Switch")
     (attr smd)
-    (fp_text reference SW1 (at 0.1545 2.296) (layer F.SilkS)
+    (fp_text reference SW1 (at 0.1545 0.0735) (layer F.SilkS)
       (effects (font (size 1 1) (thickness 0.15)))
     )
@@
     (pad 1 thru_hole circle (at 0 0) (size 2.5 2.5) (drill 2.5) (layers))
   )
+  (gr_text "IR OUT x 4" (at 144.7165 70.104) (layer F.SilkS)
+    (effects (font (size 1 1) (thickness 0.25)))
+  )
+  (gr_text GPIO (at 127.0635 66.7385 90) (layer F.SilkS)
+    (effects (font (size 1 1) (thickness 0.25)))
+  )
+  (gr_text GPIO (at 128.3335 82.2325) (layer F.SilkS)
+    (effects (font (size 1 1) (thickness 0.25)))
+  )
+  (gr_text GND (at 143.51 57.2135 360) (layer F.SilkS)
+    (effects (font (size 1 1) (thickness 0.25)))
+  )
+  (gr_text +3.3 (at 147.066 57.277) (layer F.SilkS)
+    (effects (font (size 1 1) (thickness 0.25)))
+  )
+  (gr_text GND (at 131.5085 57.9755 90) (layer F.SilkS)
+    (effects (font (size 1 1) (thickness 0.25)))
+  )
+  (gr_text LIGHT (at 115.8875 52.8955) (layer F.SilkS)
+    (effects (font (size 1 1) (thickness 0.25)))
+  )
+  (gr_text GND (at 117.983 57.277) (layer F.SilkS)
+    (effects (font (size 1 1) (thickness 0.25)))
+  )
+  (gr_text +3.3 (at 121.9835 57.404) (layer F.SilkS)
+    (effects (font (size 1 1) (thickness 0.25)))
+  )
+  (gr_text RX (at 129.032 57.404 90) (layer F.SilkS)
+    (effects (font (size 1 1) (thickness 0.25)))
+  )
+  (gr_text TX (at 126.365 57.277 90) (layer F.SilkS)
+    (effects (font (size 1 1) (thickness 0.25)))
+  )
+  (gr_text TEMP (at 136.271 52.959) (layer F.SilkS)
+    (effects (font (size 1 1) (thickness 0.25)))
+  )
+  (gr_text "IR IN" (at 141.732 52.8955) (layer F.SilkS)
+    (effects (font (size 1 1) (thickness 0.25)))
+  )
+  (gr_text GND (at 159.8295 82.1055) (layer F.SilkS)
+    (effects (font (size 1 1) (thickness 0.25)))
+  )
+  (gr_text +5 (at 162.687 82.2325) (layer F.SilkS)
+    (effects (font (size 1 1) (thickness 0.25)))
+  )
+  (gr_text PROG (at 152.2095 82.1055) (layer F.SilkS)
+    (effects (font (size 1.5 1.5) (thickness 0.3)))
+  )
+  (gr_text RESET (at 143.637 82.042) (layer F.SilkS)
+    (effects (font (size 1.5 1.5) (thickness 0.3)))
+  )
   (gr_text "IRRemote - me@pjr.cc\nhttps://github.com/takigama\n" (at 151.765 70.8025 30) (layer B.SilkS)

Commit message: updated a few bits of text on board
Other:
- board text added: "D10"
- board text added: "D13"
- board text added: "D14"
- board text added: "D16"
- board text added: "D9"
- board text added: "SPI"
Changed lines of the file:
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@@
     (links 95)
     (no_connects 0)
-    (area 100.024999 47.534523 180.387584 87.6525)
+    (area 106.424999 51.424999 175.075001 83.575001)
     (thickness 1.6)
-    (drawings 22)
+    (drawings 27)
     (tracks 455)
     (zones 0)
@@
     (pad 1 thru_hole circle (at 0 0) (size 2.5 2.5) (drill 2.5) (layers))
   )
+  (gr_text D16 (at 122.428 82.1055) (layer F.SilkS)
+    (effects (font (size 0.75 0.75) (thickness 0.1875)))
+  )
+  (gr_text D14 (at 125.0315 82.1055) (layer F.SilkS)
+    (effects (font (size 0.75 0.75) (thickness 0.1875)))
+  )
+  (gr_text D13 (at 127.5715 82.1055) (layer F.SilkS)
+    (effects (font (size 0.75 0.75) (thickness 0.1875)))
+  )
+  (gr_text D9 (at 132.6515 82.1055) (layer F.SilkS)
+    (effects (font (size 0.75 0.75) (thickness 0.1875)))
+  )
+  (gr_text D10 (at 130.175 82.1055) (layer F.SilkS)
+    (effects (font (size 0.75 0.75) (thickness 0.1875)))
+  )
   (gr_text "IR OUT x 4" (at 144.7165 70.104) (layer F.SilkS)
     (effects (font (size 1 1) (thickness 0.25)))
   )
-  (gr_text GPIO (at 127.0635 66.7385 90) (layer F.SilkS)
+  (gr_text SPI (at 127.0635 66.7385 90) (layer F.SilkS)
     (effects (font (size 1 1) (thickness 0.25)))
   )
-  (gr_text GPIO (at 128.3335 82.2325) (layer F.SilkS)
+  (gr_text GPIO (at 127.5715 77.7875) (layer F.SilkS)
     (effects (font (size 1 1) (thickness 0.25)))
   )
