File: Tasmota-Micro/Hardware/tmicro-cache.kicad_pcb (KiCad board)
At the start: 2 copper layers, 36.6 x 17.8 mm, 16 parts, among them P2 CONN_01X02, P3 CONN_01X02, P4 CONN_01X04, P5 CONN_01X02, P6 CONN_01X02, P7 USB_A, Q1 IRLML6244, Q2 IRLML6244, U1 AP1117, U2 ESP-01v090

Commit message: utas update
Parts:
- C1, C3: value 10uf -> 2uf; footprint Capacitors_SMD:C_1210 -> Capacitors_SMD:C_0805
- P7: footprint Connect:USB_A -> USB_oshpark:USB_A_Multicomp_thruhole_oshpark
- R3: moved to B.Cu
- U1: value AP1117 -> MCP1703; footprint TO_SOT_Packages_SMD:SOT-223 -> TO_SOT_Packages_SMD:SOT-23
- moved P2 11.2 mm to (167.3, 110.2)
- moved P5 11.2 mm to (160.8, 110.2)
- moved P4 11.1 mm to (160.5, 118.8)
- moved Q1 6.53 mm to (169.0, 114.2), turned to 0 degrees
- moved C1 6.06 mm to (165.8, 114.2), turned to 270 degrees
- moved R2 4.81 mm to (174.8, 114.2), turned to 270 degrees
- moved P3 4.03 mm to (175.6, 118.8)
- moved R1 3.89 mm to (172.2, 114.2), turned to 270 degrees
- moved D1 3.53 mm to (175.6, 114.2)
- moved P6 3.42 mm to (173.8, 110.2)
- moved P7 3.37 mm to (182.9, 114.5), turned to 0 degrees
- moved U1 3.26 mm to (162.6, 114.2)
- moved R3 2.37 mm to (159.4, 114.3), turned to 270 degrees
- moved Q2 2.32 mm to (177.9, 114.2), turned to 0 degrees
- moved C3 2.12 mm to (159.4, 114.2)
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Routing:
- net GND: track 61.2 -> 11.4 mm, vias 0 -> 4
- net +3V3: track 24.6 -> 4.73 mm, vias 0 -> 1
- net RX: track 30.0 -> 16.1 mm, vias 2 -> 0
- net TX: track 11.3 -> 23.1 mm
- net GPIO0: track 12.6 -> 5.54 mm
- net GPIO2: track 28.3 -> 31.0 mm, vias 1 -> 0
- net GPIO2_V: track 5.50 -> 3.98 mm
- net Net-(D1-Pad2): track 4.71 -> 5.76 mm
- net RX_V: track 5.03 -> 4.01 mm
- net VPP: track 14.7 -> 15.1 mm, vias 1 -> 0
- removed copper zone on B.Cu, net +3V3
- removed copper zone on F.Cu, net GND
- removed copper zone on B.Cu, net VPP
Other:
- board size 36.6 x 17.8 mm -> 33.5 x 13 mm
- net class 33v added: clearance 0.2, trace_width 0.4, via_dia 0.6, via_drill 0.4
- board text removed: "GND"
