File: Tasmota-Micro/Hardware/tmicro-cache.sch (KiCad schematic (older format))
At the start: 16 parts, among them P2 CONN_01X02, P3 CONN_01X02, P4 CONN_01X04, P5 CONN_01X02, P6 CONN_01X02, P7 USB_A, Q1 IRLML6244, Q2 IRLML6244, U1 AP1117, U2 ESP-01v090

Commit message: utas update
Parts:
- C1, C3: value 10uf -> 2uf; footprint Capacitors_SMD:C_1210 -> Capacitors_SMD:C_0805
- P7: footprint Connect:USB_A -> USB_oshpark:USB_A_Multicomp_thruhole_oshpark
- U1: value AP1117 -> MCP1703; footprint TO_SOT_Packages_SMD:SOT-223 -> TO_SOT_Packages_SMD:SOT-23
Changed lines of the file:
@@
 P 2950 2100
 F 0 "C3" H 2975 2200 50  0000 L CNN
-F 1 "10uf" H 2975 2000 50  0000 L CNN
-F 2 "Capacitors_SMD:C_1210" H 2988 1950 50  0001 C CNN
+F 1 "2uf" H 2975 2000 50  0000 L CNN
+F 2 "Capacitors_SMD:C_0805" H 2988 1950 50  0001 C CNN
 F 3 "" H 2950 2100 50  0000 C CNN
 F 4 "Any cap in the 0.1-10uf range" H 2950 2100 60  0001 C CNN "Notes"
@@
 P 1750 2100
 F 0 "C1" H 1775 2200 50  0000 L CNN
-F 1 "10uf" H 1775 2000 50  0000 L CNN
-F 2 "Capacitors_SMD:C_1210" H 1788 1950 50  0001 C CNN
+F 1 "2uf" H 1775 2000 50  0000 L CNN
+F 2 "Capacitors_SMD:C_0805" H 1788 1950 50  0001 C CNN
 F 3 "" H 1750 2100 50  0000 C CNN
 F 4 "a  cap of around 0.1 to 10 uf - anything in that range will do" H 1750 2100 60  0001 C CNN "Comments"
@@
 F 0 "P7" H 7350 4500 50  0000 C CNN
 F 1 "USB_A" H 7100 4900 50  0000 C CNN
-F 2 "Connect:USB_A" V 7100 4600 50  0001 C CNN
+F 2 "USB_oshpark:USB_A_Multicomp_thruhole_oshpark" V 7100 4600 50  0001 C CNN
 F 3 "" V 7100 4600 50  0000 C CNN
 	1    7150 4700
@@
 P 2350 1850
 F 0 "U1" H 2450 1600 50  0000 C CNN
-F 1 "AP1117" H 2350 2100 50  0000 C CNN
-F 2 "TO_SOT_Packages_SMD:SOT-223" H 2350 1850 50  0001 C CNN
+F 1 "MCP1703" H 2350 2100 50  0000 C CNN
+F 2 "TO_SOT_Packages_SMD:SOT-23" H 2350 1850 50  0001 C CNN
 F 3 "" H 2350 1850 50  0000 C CNN
 	1    2350 1850
