File: Tasmota-UltraMicro/Hardware/tmicro.kicad_pcb (KiCad board)
At the start: 2 copper layers, 28.1 x 11.6 mm, 10 parts, among them P1 CONN_01X04, P2 CONN_01X04, P4 CONN_01X04, P7 USB_A, U1 MCP1703, U2 ESP-01v090

Commit message: Updated ultra micro
Parts:
- moved C1 2.60 mm to (168.4, 114.6)
- moved U1 1.66 mm to (164.2, 114.4)
- moved C3 0.73 mm to (160.0, 114.4)
- moved D1 0.61 mm to (166.4, 114.4)
- moved R3 0.60 mm to (160.0, 114.3)
- moved P4 0.40 mm to (149.2, 110.6)
- moved P7 0.40 mm to (173.8, 114.4)
- moved P1 0.30 mm to (160.0, 110.2)
- moved U2 0.22 mm to (153.4, 110.6)
- moved P2 0.14 mm to (167.6, 118.6)
Routing:
- net GND: track 0.00 -> 45.2 mm
- net +3V3: track 0.00 -> 40.5 mm
- net VPP: track 0.00 -> 13.5 mm, vias 0 -> 1
- net GPIO2: track 0.00 -> 10.9 mm
- net TX: track 0.00 -> 9.36 mm
- net GPIO0: track 0.00 -> 9.35 mm
- net RX: track 0.00 -> 7.25 mm
- net Net-(R3-Pad1): track 0.00 -> 7.06 mm
- net Net-(D1-Pad2): track 0.00 -> 4.92 mm
- added copper zone on F.Cu, net GND
- added copper zone on B.Cu, net Net-(D1-Pad2)
- added copper zone on B.Cu, net VPP
Other:
- board size 28.1 x 11.6 mm -> 29 x 12.8 mm
- board text added: "GND"
- board text added: "RX"
- board text added: "TX"
- board text removed: "uTasmota v0.1 takigama@github"
